File: StackDriver/board.sch (EAGLE design)
At the start: 49 parts, among them IC1 LM741P, IC10 LM741P, IC11 LM741P, IC12 LM741P, IC13 LM741P, IC14 LM741P, IC15 LM741P, IC2 LM741P, IC3 LM741P, IC4 LM741P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

Commit message: Nie umiem w płytki. Teraz bedzie gut
Connections:
- net N$2: now also IC1.-IN; no longer IC1.+IN
- net SYG: now also IC1.+IN; no longer IC1.-IN
Changed lines of the file:
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@@
 <net name="N$2" class="0">
 <segment>
-<pinref part="IC1" gate="A" pin="+IN"/>
-<wire x1="12.7" y1="83.82" x2="2.54" y2="83.82" width="0.1524" layer="91"/>
-<wire x1="2.54" y1="83.82" x2="2.54" y2="76.2" width="0.1524" layer="91"/>
-<junction x="2.54" y="83.82"/>
 <pinref part="R2" gate="G$1" pin="1"/>
-<wire x1="2.54" y1="83.82" x2="2.54" y2="96.52" width="0.1524" layer="91"/>
+<wire x1="2.54" y1="76.2" x2="2.54" y2="78.74" width="0.1524" layer="91"/>
+<wire x1="2.54" y1="78.74" x2="2.54" y2="96.52" width="0.1524" layer="91"/>
 <wire x1="2.54" y1="96.52" x2="15.24" y2="96.52" width="0.1524" layer="91"/>
 <pinref part="R1" gate="G$1" pin="2"/>
+<pinref part="IC1" gate="A" pin="-IN"/>
+<wire x1="12.7" y1="78.74" x2="2.54" y2="78.74" width="0.1524" layer="91"/>
+<junction x="2.54" y="78.74"/>
 </segment>
 </net>
 <net name="SYG" class="0">
-<segment>
-<pinref part="IC1" gate="A" pin="-IN"/>
-<wire x1="12.7" y1="78.74" x2="-10.16" y2="78.74" width="0.1524" layer="91"/>
-<junction x="-10.16" y="78.74"/>
-<label x="-10.16" y="78.74" size="1.778" layer="95"/>
-</segment>
 <segment>
 <pinref part="IC2" gate="A" pin="-IN"/>
@@
 <label x="-58.42" y="81.28" size="1.778" layer="95"/>
 </segment>
+<segment>
+<pinref part="IC1" gate="A" pin="+IN"/>
+<wire x1="12.7" y1="83.82" x2="-5.08" y2="83.82" width="0.1524" layer="91"/>
+<junction x="-5.08" y="83.82"/>
+<label x="-5.08" y="83.82" size="1.778" layer="95"/>
+</segment>
 </net>
