File: StackDriver 2.0/driverV3.brd (EAGLE design)
At the start: 100 x 80 mm, 46 parts, among them U1 NE5532N, U2 NE5532N, U3 NE5532N, U4 NE5532N, U5 NE5532N, U6 NE5532N, U7 NE5532N, U8 NE5532N

Commit message: chyba działa
Parts:
- moved R29 126.9 mm to (62.2, 19.1)
- moved JP2 125.1 mm to (86.4, 61.0), turned to 90 degrees
- moved R28 121.4 mm to (68.6, 25.4), turned to 90 degrees
- moved R4 120.1 mm to (53.3, 73.7), turned to 270 degrees
- moved R8 119.1 mm to (68.6, 61.0), turned to 90 degrees
- moved U2 117.7 mm to (64.8, 73.7), flipped to the bottom
- moved U8 114.5 mm to (57.1, 25.4), flipped to the bottom, turned to 180 degrees
- moved R3 113.0 mm to (55.9, 73.7), turned to 270 degrees
- moved U7 110.9 mm to (64.8, 38.1), flipped to the bottom
- moved R27 109.2 mm to (66.0, 25.4), turned to 90 degrees
- moved U4 106.8 mm to (33.0, 63.5), flipped to the bottom
- moved R7 106.6 mm to (66.0, 61.0), turned to 90 degrees
- moved R6 104.5 mm to (66.0, 83.8), turned to 90 degrees
- moved R19 98.4 mm to (34.3, 15.2), turned to 90 degrees
- moved R14 97.6 mm to (34.3, 73.7), turned to 90 degrees
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Connections:
- removed net V+: U1.8, U2.8, U3.8, U4.8, U5.8, U6.8, U7.8, U8.8
- removed net V-: U1.4, U2.4, U3.4, U4.4, U5.4, U6.4, U7.4, U8.4
- net 1: now also R12.2, U3.1; no longer R4.2, U1.1
- net 10: now also R2.1, U1.7; no longer R18.1, U5.7
- net 13: now also R28.2, U7.1; no longer R12.2, U3.1
- net 14: now also R26.1, U7.7; no longer R10.1, U3.7
- net 15: now also R8.2, U2.1; no longer R24.2, U6.1
- net 16: now also R6.1, U2.7; no longer R22.1, U6.7
- net 2: now also R10.1, U3.7; no longer R2.1, U1.7
- net 3: now also R24.2, U6.1; no longer R16.2, U4.1
- net 4: now also R22.1, U6.7; no longer R14.1, U4.7
- net 5: now also R20.2, U5.1; no longer R28.2, U7.1
- net 6: now also R18.1, U5.7; no longer R26.1, U7.7
- net 7: now also R16.2, U4.1; no longer R8.2, U2.1
- net 8: now also R14.1, U4.7; no longer R6.1, U2.7
- net 9: now also R4.2, U1.1; no longer R20.2, U5.1
- net GND: now also U1.4, U2.4, U3.4, U4.4, U5.4, U6.4, U7.4, U8.4
- net VCC: now also U1.8, U2.8, U3.8, U4.8, U5.8, U6.8, U7.8, U8.8
Routing:
- net GND: track 0.00 -> 321.8 mm
- net SYG: track 0.00 -> 134.5 mm
- net 1: track 0.00 -> 120.4 mm
- net 2: track 0.00 -> 100.4 mm
- net 8: track 0.00 -> 92.2 mm
- net 9: track 0.00 -> 87.6 mm
- net 3: track 0.00 -> 78.3 mm
- net 7: track 0.00 -> 77.7 mm
- net VCC: track 0.00 -> 76.5 mm, vias 0 -> 8
- net 10: track 0.00 -> 67.6 mm
- net 6: track 0.00 -> 59.1 mm
- net 5: track 0.00 -> 48.6 mm
- net 4: track 0.00 -> 48.0 mm
- net 11: track 0.00 -> 45.5 mm
- net 14: track 0.00 -> 42.9 mm
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Other:
- board size 100 x 80 mm -> 100 x 91.4 mm
