File: StackDriver 2.0/driverV3.sch (EAGLE design)
At the start: 46 parts, among them U1 NE5532N, U2 NE5532N, U3 NE5532N, U4 NE5532N, U5 NE5532N, U6 NE5532N, U7 NE5532N, U8 NE5532N

Commit message: chyba działa
Connections:
- net 1: now also R12.2, U3A.OUT; no longer R4.2, U1A.OUT
- net 10: now also R2.1, U1B.OUT; no longer R18.1, U5B.OUT
- net 13: now also R28.2, U7A.OUT; no longer R12.2, U3A.OUT
- net 14: now also R26.1, U7B.OUT; no longer R10.1, U3B.OUT
- net 15: now also R8.2, U2A.OUT; no longer R24.2, U6A.OUT
- net 16: now also R6.1, U2B.OUT; no longer R22.1, U6B.OUT
- net 2: now also R10.1, U3B.OUT; no longer R2.1, U1B.OUT
- net 3: now also R24.2, U6A.OUT; no longer R16.2, U4A.OUT
- net 4: now also R22.1, U6B.OUT; no longer R14.1, U4B.OUT
- net 5: now also R20.2, U5A.OUT; no longer R28.2, U7A.OUT
- net 6: now also R18.1, U5B.OUT; no longer R26.1, U7B.OUT
- net 7: now also R16.2, U4A.OUT; no longer R8.2, U2A.OUT
- net 8: now also R14.1, U4B.OUT; no longer R6.1, U2B.OUT
- net 9: now also R4.2, U1A.OUT; no longer R20.2, U5A.OUT
